Commit message: description changes

File: narval_description/xacro/bluerov2.urdf.xacro (robot description, xacro)
@@ -23,8 +23,11 @@
   <xacro:property name="LENGTH" value="0.662"/>
   <xacro:property name="MASS" value="11.51"/>
-  <xacro:property name="CoG_X" value="0.03435"/>
-  <xacro:property name="CoG_Y" value="0.001402"/>
-  <xacro:property name="CoG_Z" value="0.00012"/>
+  <xacro:property name="CoG_X" value="0"/>
+  <xacro:property name="CoG_Y" value="0"/>
+  <xacro:property name="CoG_Z" value="0.05"/>
   <xacro:property name="CoG" value="${CoG_X} ${CoG_Y} ${CoG_Z}"/>
+  <xacro:macro name='CoG_origin' params="X Y Z rpy" >
+    <origin xyz="${X + CoG_X} ${Y + CoG_Y} ${Z + CoG_Z}" rpy="${rpy}"/>
+  </xacro:macro>
   <!-- Thruster macro -->
   <xacro:macro name="t200" params="side name *origin">
@@ -45,5 +48,6 @@
   <link name="base_link">
     <visual>
-      <origin xyz="0.0 0.0 0.0" rpy="${PI} 0.0 0.0"/>
+      <!-- <origin xyz="0.0 0.0 0.0" rpy="${PI} 0.0 0.0"/> -->
+      <xacro:CoG_origin X="0" Y="0" Z="0" rpy="${PI} 0 0"/>
       <geometry>
         <mesh filename="package://narval_description/meshes/bluerov2.obj" scale="1 1 1"/>
@@ -52,5 +56,6 @@
     </visual>
     <collision>
-      <origin xyz="0.0 0.0 0.0" rpy="${PI} 0.0 0.0"/>
+      <!-- <origin xyz="0.0 0.0 0.0" rpy="${PI} 0.0 0.0"/> -->
+      <xacro:CoG_origin X="0" Y="0" Z="0" rpy="${PI} 0 0"/>
       <geometry>
         <mesh filename="package://narval_description/meshes/bluerov2_phy.obj" scale="1 1 1"/>
@@ -58,5 +63,6 @@
     </collision>
     <visual>
-      <origin xyz="0.0 0.0 0.03" rpy="${PI} 0.0 0.0"/>
+      <!-- <origin xyz="0.0 0.0 0.03" rpy="${PI} 0.0 0.0"/> -->
+      <xacro:CoG_origin X="0" Y="0" Z="0.03" rpy="${PI} 0 0"/>
       <geometry>
         <mesh filename="package://narval_description/meshes/bluerov2_wings.obj" scale="1 1 1"/>
@@ -65,5 +71,6 @@
     </visual>
     <collision>
-      <origin xyz="0.0 0.0 0.03" rpy="${PI} 0.0 0.0"/>
+      <!-- <origin xyz="0.0 0.0 0.03" rpy="${PI} 0.0 0.0"/> -->
+      <xacro:CoG_origin X="0" Y="0" Z="0.03" rpy="${PI} 0 0"/>
       <geometry>
         <mesh filename="package://narval_description/meshes/bluerov2_ring.obj" scale="1 1 1"/>
@@ -74,33 +81,41 @@
   <xacro:property name="front_right_origin">
     <!-- <origin xyz="0.1355 0.1 0.0725" rpy="0 0 -0.7853981634"/> -->
-    <origin xyz="0.1355 0.1 -0.0725" rpy="${PI} 0 -0.7853981634"/>
+    <!-- <origin xyz="0.1355 0.1 -0.0725" rpy="${PI} 0 -0.7853981634"/> -->
+    <xacro:CoG_origin X="0.1355" Y="0.1" Z="-0.0725" rpy="0 0 -0.7853981634"/>
   </xacro:property>
   <xacro:property name="front_left_origin">
     <!-- <origin xyz="0.1355 -0.1 0.0725" rpy="0 0 0.7853981634"/> -->
-    <origin xyz="0.1355 -0.1 -0.0725" rpy="${PI} 0 0.7853981634"/>
+    <!-- <origin xyz="0.1355 -0.1 -0.0725" rpy="${PI} 0 0.7853981634"/> -->
+    <xacro:CoG_origin X="0.1355" Y="-0.1" Z="-0.0725" rpy="0 0 0.7853981634"/>
   </xacro:property>
   <xacro:property name="rear_right_origin">
     <!-- <origin xyz="-0.1475 0.1 0.0725" rpy="0 0 -2.3561944902"/> -->
-    <origin xyz="-0.1475 0.1 -0.0725" rpy="${PI} 0 -2.3561944902"/>
+    <!-- <origin xyz="-0.1475 0.1 -0.0725" rpy="${PI} 0 -2.3561944902"/> -->
+    <xacro:CoG_origin X="-0.1475" Y="0.1" Z="-0.0725" rpy="0 0 -2.3561944902"/>
   </xacro:property>
   <xacro:property name="rear_left_origin">
     <!-- <origin xyz="-0.1475 -0.1 0.0725" rpy="0 0 2.3561944902"/> -->
-    <origin xyz="-0.1475 -0.1 -0.0725" rpy="${PI} 0 2.3561944902"/>
+    <!-- <origin xyz="-0.1475 -0.1 -0.0725" rpy="${PI} 0 2.3561944902"/> -->
+    <xacro:CoG_origin X="-0.1475" Y="-0.1" Z="-0.0725" rpy="0 0 2.3561944902"/>
   </xacro:property>
   <xacro:property name="dive_front_right_origin">
     <!-- <origin xyz="0.12 0.218 0.0" rpy="0 -1.5707963268 0"/> -->
-    <origin xyz="0.12 0.218 0.0" rpy="${PI} -1.5707963268 0"/>
+    <!-- <origin xyz="0.12 0.218 0.0" rpy="${PI} -1.5707963268 0"/> -->
+    <xacro:CoG_origin X="0.12" Y="0.218" Z="0.0" rpy="${PI} -1.5707963268 0"/>
   </xacro:property>
   <xacro:property name="dive_front_left_origin">
     <!-- <origin xyz="0.12 -0.218 0.0" rpy="0 -1.5707963268 0"/> -->
-    <origin xyz="0.12 -0.218 0.0" rpy="${PI} -1.5707963268 0"/>
+    <!-- <origin xyz="0.12 -0.218 0.0" rpy="${PI} -1.5707963268 0"/> -->
+    <xacro:CoG_origin X="0.12" Y="-0.218" Z="0.0" rpy="${PI} -1.5707963268 0"/>
   </xacro:property>
   <xacro:property name="dive_rear_right_origin">
     <!-- <origin xyz="-0.12 0.218 0.0" rpy="0 -1.5707963268 0"/> -->
-    <origin xyz="-0.12 0.218 0.0" rpy="${PI} -1.5707963268 0"/>
+    <!-- <origin xyz="-0.12 0.218 0.0" rpy="${PI} -1.5707963268 0"/> -->
+    <xacro:CoG_origin X="-0.12" Y="0.218" Z="0.0" rpy="${PI} -1.5707963268 0"/>
   </xacro:property>
   <xacro:property name="dive_rear_left_origin">
     <!-- <origin xyz="-0.12 -0.218 0.0" rpy="0 -1.5707963268 0"/> -->
-    <origin xyz="-0.12 -0.218 0.0" rpy="${PI} -1.5707963268 0"/>
+    <!-- <origin xyz="-0.12 -0.218 0.0" rpy="${PI} -1.5707963268 0"/> -->
+    <xacro:CoG_origin X="-0.12" Y="-0.218" Z="0.0" rpy="${PI} -1.5707963268 0"/>
   </xacro:property>
   <!-- Attach thrusters to the base_link -->

File: narval_description/xacro/narval_base.urdf.xacro (robot description, xacro)
@@ -112,20 +112,20 @@
     </link>
     <!-- Attach thrusters to the base_link -->
-    <xacro:t200 name="front_right" side="right">
+    <xacro:t200 name="t1" side="right">
         <xacro:insert_block name="front_right_origin" />
     </xacro:t200>
-    <xacro:t200 name="front_left" side="left">
+    <xacro:t200 name="t2" side="left">
         <xacro:insert_block name="front_left_origin" />
     </xacro:t200>
-    <xacro:t200 name="rear_right" side="right">
+    <xacro:t200 name="t5" side="right">
         <xacro:insert_block name="rear_right_origin" />
     </xacro:t200>
-    <xacro:t200 name="rear_left" side="left">
+    <xacro:t200 name="t6" side="left">
         <xacro:insert_block name="rear_left_origin" />
     </xacro:t200>
-    <xacro:t200 name="middle_right" side="right">
+    <xacro:t200 name="t3" side="right">
         <xacro:insert_block name="middle_right_origin" />
     </xacro:t200>
-    <xacro:t200 name="middle_left" side="left">
+    <xacro:t200 name="t4" side="left">
         <xacro:insert_block name="middle_left_origin" />
     </xacro:t200>
